File: sequint.sch (EAGLE design)
At the start: 72 parts, among them IC1 STM32F10XCXT6, Q1 MOSFET-NCHANNELSMD, Q2 MOSFET-NCHANNELSMD, Q3 MOSFET-NCHANNELSMD, Q4 MOSFET-NCHANNELSMD, Q5 16MHz, U1 LSM330DLCTRLGA, U2 MCP73831, U4 NRF24L01SMD

Commit message: Move USART to USART1, which supports bootloader.
Connections:
- new net PB4: IC1PORTB_L.PB4, JP1.1
- new net PB5: IC1PORTB_L.PB5, JP1.2
- new net PB9: IC1PORTB_H.PB9, JP1.3
- net 5V-SENSE: now also IC1PORTB_H.PB11; no longer IC1PORTA_H.PA9
- net LIPO-STAT: now also IC1PORTB_H.PB10; no longer IC1PORTA_H.PA10
- net RX: now also IC1PORTA_H.PA10; no longer IC1PORTB_H.PB11
- net TX: now also IC1PORTA_H.PA9; no longer IC1PORTB_H.PB10
Other:
- moved on the sheet: JP1
Changed lines of the file:
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@@
 <instance part="LED1" gate="G$1" x="83.82" y="38.1"/>
 <instance part="R10" gate="G$1" x="63.5" y="43.18"/>
-<instance part="JP1" gate="A" x="-40.64" y="27.94"/>
+<instance part="JP1" gate="A" x="124.46" y="71.12"/>
 </instances>
 <busses>
@@
 <segment>
 <pinref part="JP1" gate="A" pin="4"/>
-<wire x1="-43.18" y1="25.4" x2="-50.8" y2="25.4" width="0.1524" layer="91"/>
-<label x="-53.34" y="25.4" size="1.778" layer="95"/>
+<wire x1="121.92" y1="68.58" x2="114.3" y2="68.58" width="0.1524" layer="91"/>
+<label x="111.76" y="68.58" size="1.778" layer="95"/>
 </segment>
 </net>
@@
 <net name="TX" class="0">
 <segment>
-<label x="33.02" y="71.12" size="1.778" layer="95"/>
+<label x="55.88" y="71.12" size="1.778" layer="95"/>
 <pinref part="SERIAL" gate="A" pin="1"/>
-<pinref part="IC1" gate="PORTB_H" pin="PB10"/>
-<wire x1="30.48" y1="71.12" x2="63.5" y2="71.12" width="0" layer="91"/>
+<wire x1="63.5" y1="71.12" x2="55.88" y2="71.12" width="0.1524" layer="91"/>
+</segment>
+<segment>
+<pinref part="IC1" gate="PORTA_H" pin="PA9"/>
+<wire x1="-5.08" y1="73.66" x2="-7.62" y2="73.66" width="0.1524" layer="91"/>
+<label x="-7.62" y="73.66" size="1.778" layer="95" rot="R180"/>
 </segment>
 </net>
 <net name="RX" class="0">
 <segment>
-<label x="33.02" y="68.58" size="1.778" layer="95"/>
+<label x="55.88" y="68.58" size="1.778" layer="95"/>
 <pinref part="SERIAL" gate="A" pin="2"/>
-<pinref part="IC1" gate="PORTB_H" pin="PB11"/>
-<wire x1="30.48" y1="68.58" x2="63.5" y2="68.58" width="0" layer="91"/>
+<wire x1="63.5" y1="68.58" x2="55.88" y2="68.58" width="0.1524" layer="91"/>
+</segment>
+<segment>
+<pinref part="IC1" gate="PORTA_H" pin="PA10"/>
+<wire x1="-5.08" y1="71.12" x2="-7.62" y2="71.12" width="0.1524" layer="91"/>
+<label x="-7.62" y="71.12" size="1.778" layer="95" rot="R180"/>
 </segment>
 </net>
@@
 <net name="LIPO-STAT" class="0">
 <segment>
-<label x="-7.62" y="71.12" size="1.778" layer="95" rot="R180"/>
-<pinref part="IC1" gate="PORTA_H" pin="PA10"/>
-<wire x1="-5.08" y1="71.12" x2="-7.62" y2="71.12" width="0.1524" layer="91"/>
+<label x="33.02" y="71.12" size="1.778" layer="95"/>
+<pinref part="IC1" gate="PORTB_H" pin="PB10"/>
+<wire x1="30.48" y1="71.12" x2="33.02" y2="71.12" width="0.1524" layer="91"/>
 </segment>
 </net>
@@
 <wire x1="-5.08" y1="93.98" x2="-7.62" y2="93.98" width="0" layer="91"/>
 <label x="-7.62" y="93.98" size="1.778" layer="95" rot="R180"/>
-</segment>
-</net>
-<net name="5V-SENSE" class="0">
-<segment>
-<label x="-7.62" y="73.66" size="1.778" layer="95" rot="R180"/>
-<pinref part="IC1" gate="PORTA_H" pin="PA9"/>
-<wire x1="-5.08" y1="73.66" x2="-7.62" y2="73.66" width="0.1524" layer="91"/>
 </segment>
 </net>
@@
 </segment>
 </net>
+<net name="5V-SENSE" class="0">
+<segment>
+<pinref part="IC1" gate="PORTB_H" pin="PB11"/>
+<wire x1="30.48" y1="68.58" x2="33.02" y2="68.58" width="0.1524" layer="91"/>
+<label x="33.02" y="68.58" size="1.778" layer="95"/>
+</segment>
+</net>
+<net name="PB4" class="0">
+<segment>
+<pinref part="IC1" gate="PORTB_L" pin="PB4"/>
+<wire x1="30.48" y1="93.98" x2="33.02" y2="93.98" width="0.1524" layer="91"/>
+<label x="33.02" y="93.98" size="1.778" layer="95"/>
+</segment>
+<segment>
+<pinref part="JP1" gate="A" pin="1"/>
+<wire x1="121.92" y1="76.2" x2="114.3" y2="76.2" width="0.1524" layer="91"/>
+</segment>
+</net>
+<net name="PB5" class="0">
+<segment>
+<pinref part="IC1" gate="PORTB_L" pin="PB5"/>
+<wire x1="30.48" y1="91.44" x2="33.02" y2="91.44" width="0.1524" layer="91"/>
+<label x="33.02" y="91.44" size="1.778" layer="95"/>
+</segment>
+<segment>
+<pinref part="JP1" gate="A" pin="2"/>
+<wire x1="121.92" y1="73.66" x2="114.3" y2="73.66" width="0.1524" layer="91"/>
+</segment>
+</net>
+<net name="PB9" class="0">
+<segment>
+<pinref part="IC1" gate="PORTB_H" pin="PB9"/>
+<wire x1="30.48" y1="73.66" x2="33.02" y2="73.66" width="0.1524" layer="91"/>
+<label x="33.02" y="73.66" size="1.778" layer="95"/>
+</segment>
+<segment>
+<pinref part="JP1" gate="A" pin="3"/>
+<wire x1="121.92" y1="71.12" x2="114.3" y2="71.12" width="0.1524" layer="91"/>
+</segment>
+</net>

Commit message: Silkscreen
Parts:
- IC1: value STM32F10XCXT6 -> STM32F103
- Q1, Q2, Q3, Q4: value MOSFET-NCHANNELSMD -> MOSFET-N
Changed lines of the file:
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@@
 </classes>
 <parts>
-<part name="IC1" library="stm32" deviceset="STM32F10XCXT6" device=""/>
-<part name="Q1" library="SparkFun" deviceset="MOSFET-NCHANNEL" device="SMD"/>
-<part name="Q2" library="SparkFun" deviceset="MOSFET-NCHANNEL" device="SMD"/>
-<part name="Q3" library="SparkFun" deviceset="MOSFET-NCHANNEL" device="SMD"/>
-<part name="Q4" library="SparkFun" deviceset="MOSFET-NCHANNEL" device="SMD"/>
+<part name="IC1" library="stm32" deviceset="STM32F10XCXT6" device="" value="STM32F103"/>
+<part name="Q1" library="SparkFun" deviceset="MOSFET-NCHANNEL" device="SMD" value="MOSFET-N"/>
+<part name="Q2" library="SparkFun" deviceset="MOSFET-NCHANNEL" device="SMD" value="MOSFET-N"/>
+<part name="Q3" library="SparkFun" deviceset="MOSFET-NCHANNEL" device="SMD" value="MOSFET-N"/>
+<part name="Q4" library="SparkFun" deviceset="MOSFET-NCHANNEL" device="SMD" value="MOSFET-N"/>
 <part name="JTAG" library="nonolith" deviceset="HEADER-2X5" device=""/>
 <part name="U1" library="nonolith" deviceset="LSM330DLCTR" device="LGA"/>
