File: sequint.brd (EAGLE design)
At the start: 70 x 80 mm, 72 parts, among them IC1 STM32F10XCXT6, Q1 MOSFET-NCHANNELSMD, Q2 MOSFET-NCHANNELSMD, Q3 MOSFET-NCHANNELSMD, Q4 MOSFET-NCHANNELSMD, Q5 16MHz, U1 LSM330DLCTRLGA, U2 MCP73831, U4 NRF24L01SMD

Commit message: Clean up
Routing:
- net GND: track 97.2 -> 98.2 mm, vias 42 -> 50
Changed lines of the file:
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@@
 <wire x1="19.477" y1="45.917" x2="18.161" y2="44.577" width="0.254" layer="1"/>
 <via x="14.224" y="45.974" extent="1-16" drill="0.3302"/>
-<via x="61.468" y="38.735" extent="1-16" drill="0.3302"/>
+<via x="59.944" y="38.481" extent="1-16" drill="0.3302"/>
 <via x="21.59" y="59.055" extent="1-16" drill="0.3302"/>
+<via x="20.828" y="44.323" extent="1-16" drill="0.3302"/>
+<via x="28.702" y="44.196" extent="1-16" drill="0.3302"/>
+<via x="66.802" y="33.02" extent="1-16" drill="0.3302"/>
+<via x="55.118" y="61.722" extent="1-16" drill="0.3302"/>
+<via x="20.066" y="54.61" extent="1-16" drill="0.3302"/>
+<via x="28.448" y="56.642" extent="1-16" drill="0.3302"/>
+<via x="22.733" y="69.723" extent="1-16" drill="0.3302"/>
+<wire x1="29.337" y1="50.419" x2="28.321" y2="50.419" width="0.254" layer="1"/>
+<via x="22.098" y="53.721" extent="1-16" drill="0.3302"/>
+<wire x1="29.2624" y1="50.4236" x2="29.337" y2="50.419" width="0" layer="19" extent="1-1"/>
 </signal>
 <signal name="3.3V">
@@
 <wire x1="10.033" y1="59.436" x2="10.033" y2="68.834" width="0.254" layer="1"/>
 <wire x1="10.033" y1="68.834" x2="10.287" y2="69.088" width="0.254" layer="1"/>
-<wire x1="12.545" y1="56.962" x2="19.746" y2="56.962" width="0.254" layer="1"/>
-<via x="19.746" y="56.962" extent="1-16" drill="0.3302"/>
-<wire x1="19.746" y1="56.962" x2="26.416" y2="50.292" width="0.254" layer="16"/>
+<wire x1="12.545" y1="56.962" x2="19.111" y2="56.962" width="0.254" layer="1"/>
+<via x="19.111" y="56.962" extent="1-16" drill="0.3302"/>
 <wire x1="26.416" y1="50.292" x2="26.416" y2="46.609" width="0.254" layer="16"/>
 <wire x1="26.5124" y1="43.6736" x2="26.5124" y2="46.5126" width="0.254" layer="1"/>
 <wire x1="26.5124" y1="46.5126" x2="26.416" y2="46.609" width="0.254" layer="1"/>
 <via x="26.416" y="46.609" extent="1-16" drill="0.3302"/>
+<wire x1="19.111" y1="56.962" x2="19.746" y2="56.962" width="0.254" layer="16"/>
+<wire x1="19.746" y1="56.962" x2="26.416" y2="50.292" width="0.254" layer="16"/>
 </signal>
 <signal name="TMR2-CH2">

Commit message: Clean up
Routing:
- net GND: track 98.2 -> 100.2 mm
Changed lines of the file:
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@@
 <via x="52.169" y="27.752" extent="1-16" drill="0.3302"/>
 <via x="52.169" y="28.895" extent="1-16" drill="0.3302"/>
-<wire x1="20.2624" y1="45.9236" x2="19.477" y2="45.917" width="0.254" layer="1"/>
-<wire x1="19.477" y1="45.917" x2="18.161" y2="44.577" width="0.254" layer="1"/>
 <via x="14.224" y="45.974" extent="1-16" drill="0.3302"/>
 <via x="59.944" y="38.481" extent="1-16" drill="0.3302"/>
@@
 <wire x1="29.337" y1="50.419" x2="28.321" y2="50.419" width="0.254" layer="1"/>
 <via x="22.098" y="53.721" extent="1-16" drill="0.3302"/>
+<wire x1="19.558" y1="45.974" x2="18.161" y2="44.577" width="0.254" layer="1"/>
+<wire x1="21.483" y1="45.947" x2="19.578" y2="45.947" width="0.254" layer="1"/>
+<wire x1="19.558" y1="45.974" x2="20.212" y2="45.974" width="0.254" layer="1"/>
+<wire x1="20.212" y1="45.974" x2="20.2624" y2="45.9236" width="0.254" layer="1"/>
 <wire x1="29.2624" y1="50.4236" x2="29.337" y2="50.419" width="0" layer="19" extent="1-1"/>
+<wire x1="19.578" y1="45.947" x2="19.578" y2="45.954" width="0.254" layer="1"/>
+<wire x1="19.578" y1="45.954" x2="19.558" y2="45.974" width="0.254" layer="1"/>
 </signal>
 <signal name="3.3V">

Commit message: Silkscreen
Parts:
- IC1: value STM32F10XCXT6 -> STM32F103
- Q1, Q2, Q3, Q4: value MOSFET-NCHANNELSMD -> MOSFET-N
Changed lines of the file:
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@@
 <layer number="25" name="tNames" color="7" fill="1" visible="yes" active="yes"/>
 <layer number="26" name="bNames" color="7" fill="1" visible="yes" active="yes"/>
-<layer number="27" name="tValues" color="7" fill="1" visible="yes" active="yes"/>
-<layer number="28" name="bValues" color="7" fill="1" visible="yes" active="yes"/>
-<layer number="29" name="tStop" color="7" fill="3" visible="no" active="yes"/>
+<layer number="27" name="tValues" color="7" fill="1" visible="no" active="yes"/>
+<layer number="28" name="bValues" color="7" fill="1" visible="no" active="yes"/>
+<layer number="29" name="tStop" color="7" fill="3" visible="yes" active="yes"/>
 <layer number="30" name="bStop" color="7" fill="6" visible="no" active="yes"/>
 <layer number="31" name="tCream" color="7" fill="4" visible="no" active="yes"/>
@@
 <wire x1="70" y1="80" x2="0" y2="80" width="0" layer="20"/>
 <wire x1="0" y1="80" x2="0" y2="0" width="0" layer="20"/>
-<rectangle x1="33.782" y1="2.794" x2="57.15" y2="10.922" layer="21"/>
+<rectangle x1="32.004" y1="2.667" x2="55.372" y2="10.795" layer="21"/>
 <text x="16.256" y="7.62" size="1.27" layer="21" ratio="12">Nonolith Labs</text>
 <text x="16.256" y="5.334" size="1.27" layer="21" ratio="12">μ4 roadkill 0.1</text>
@@
 </autorouter>
 <elements>
-<element name="IC1" library="stm32" package="TQFP48" value="STM32F10XCXT6" x="24.7624" y="48.1736"/>
-<element name="Q1" library="SparkFun" package="SOT23-3" value="MOSFET-NCHANNELSMD" x="4.036" y="68.011"/>
-<element name="Q2" library="SparkFun" package="SOT23-3" value="MOSFET-NCHANNELSMD" x="56.868" y="74.996" rot="R270"/>
-<element name="Q3" library="SparkFun" package="SOT23-3" value="MOSFET-NCHANNELSMD" x="66.548" y="12.192" rot="R180"/>
-<element name="Q4" library="SparkFun" package="SOT23-3" value="MOSFET-NCHANNELSMD" x="12.291" y="3.368" rot="R90"/>
+<element name="IC1" library="stm32" package="TQFP48" value="STM32F103" x="24.7624" y="48.1736" smashed="yes">
+<attribute name="NAME" x="22.2224" y="48.6816" size="1.27" layer="25"/>
+<attribute name="VALUE" x="21.8414" y="47.5386" size="0.762" layer="27"/>
+</element>
+<element name="Q1" library="SparkFun" package="SOT23-3" value="MOSFET-N" x="4.036" y="68.011"/>
+<element name="Q2" library="SparkFun" package="SOT23-3" value="MOSFET-N" x="56.868" y="74.996" rot="R270"/>
+<element name="Q3" library="SparkFun" package="SOT23-3" value="MOSFET-N" x="66.548" y="12.192" rot="R180"/>
+<element name="Q4" library="SparkFun" package="SOT23-3" value="MOSFET-N" x="12.291" y="3.368" rot="R90"/>
 <element name="JTAG" library="nonolith" package="2X05" value="" x="5.56" y="48.58" rot="R270"/>
 <element name="U1" library="nonolith" package="LGA28L" value="LSM330DLCTRLGA" x="52.042" y="28.641" rot="R90"/>
@@
 <element name="U2" library="SparkFun" package="SOT23-5" value="MCP73831" x="35.278" y="70.932"/>
 <element name="R5" library="nonolith" package="0402" value="10ko" x="32.992" y="65.598" rot="R270"/>
-<element name="3.3VREG" library="nonolith" package="SOT23-3" value="VREG" x="47.978" y="66.614" rot="R180"/>
-<element name="C7" library="nonolith" package="0603" value="4.7uF" x="43.914" y="65.344"/>
+<element name="3.3VREG" library="nonolith" package="SOT23-3" value="VREG" x="47.978" y="66.614" smashed="yes" rot="R180">
+<attribute name="VALUE" x="49.883" y="70.043" size="1.27" layer="27" rot="R180"/>
+</element>
+<element name="C7" library="nonolith" package="0603" value="4.7uF" x="43.914" y="65.344" smashed="yes">
+<attribute name="NAME" x="44.168" y="63.693" size="0.762" layer="25" font="vector" ratio="10"/>
+</element>
 <element name="Q5" library="nonolith" package="HC49UP" value="16MHz" x="54.2518" y="46.8782"/>
 <element name="L1" library="SparkFun" package="C0402" value="3.9nH" x="58.1126" y="55.0062" rot="R90"/>

Commit message: fix airwires
Routing:
- net GND: track 100.2 -> 103.9 mm
Changed lines of the file:
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@@
 <layer number="27" name="tValues" color="7" fill="1" visible="no" active="yes"/>
 <layer number="28" name="bValues" color="7" fill="1" visible="no" active="yes"/>
-<layer number="29" name="tStop" color="7" fill="3" visible="yes" active="yes"/>
+<layer number="29" name="tStop" color="7" fill="3" visible="no" active="yes"/>
 <layer number="30" name="bStop" color="7" fill="6" visible="no" active="yes"/>
 <layer number="31" name="tCream" color="7" fill="4" visible="no" active="yes"/>
@@
 <wire x1="19.558" y1="45.974" x2="20.212" y2="45.974" width="0.254" layer="1"/>
 <wire x1="20.212" y1="45.974" x2="20.2624" y2="45.9236" width="0.254" layer="1"/>
-<wire x1="29.2624" y1="50.4236" x2="29.337" y2="50.419" width="0" layer="19" extent="1-1"/>
 <wire x1="19.578" y1="45.947" x2="19.578" y2="45.954" width="0.254" layer="1"/>
 <wire x1="19.578" y1="45.954" x2="19.558" y2="45.974" width="0.254" layer="1"/>
+<wire x1="29.2624" y1="50.4236" x2="27.178" y2="50.4236" width="0.254" layer="1"/>
+<wire x1="27.178" y1="50.4236" x2="27.178" y2="50.673" width="0.254" layer="1"/>
+<wire x1="27.178" y1="50.673" x2="28.321" y2="50.673" width="0.254" layer="1"/>
+<wire x1="28.321" y1="50.673" x2="28.321" y2="50.419" width="0.254" layer="1"/>
 </signal>
 <signal name="3.3V">
@@
 <wire x1="55.179" y1="28.133" x2="56.614" y2="28.133" width="0.254" layer="16"/>
 <wire x1="51.181" y1="33.909" x2="50.546" y2="34.544" width="0.254" layer="1"/>
-<wire x1="50.546" y1="34.544" x2="50.546" y2="36.068" width="0.254" layer="1"/>
+<wire x1="50.546" y1="34.544" x2="50.546" y2="36.18" width="0.254" layer="1"/>
 <wire x1="56.614" y1="28.133" x2="56.802" y2="28.321" width="0.254" layer="1"/>
 <wire x1="56.802" y1="28.321" x2="58.039" y2="28.321" width="0.254" layer="1"/>
@@
 <wire x1="22.832" y1="61.646" x2="21.666" y2="61.646" width="0.254" layer="1"/>
 <wire x1="21.666" y1="61.646" x2="18.542" y2="64.77" width="0.254" layer="1"/>
-<wire x1="18.542" y1="64.77" x2="17.653" y2="64.77" width="0.254" layer="1"/>
-<wire x1="50.546" y1="36.068" x2="50.546" y2="36.18" width="0" layer="19" extent="1-1"/>
-<wire x1="17.78" y1="64.77" x2="17.653" y2="64.77" width="0" layer="19" extent="1-1"/>
+<wire x1="17.78" y1="64.77" x2="18.542" y2="64.77" width="0.254" layer="1"/>
 </signal>
 <signal name="USB-DM">
@@
 <contactref element="JTAG" pad="10"/>
 <contactref element="IC1" pad="7"/>
-<wire x1="15.748" y1="43.434" x2="15.621" y2="43.434" width="0.254" layer="16"/>
-<wire x1="15.621" y1="43.434" x2="6.858" y2="43.434" width="0.254" layer="16"/>
+<wire x1="23.622" y1="43.434" x2="6.83" y2="43.434" width="0.254" layer="16"/>
 <wire x1="25.0124" y1="43.6736" x2="25.0124" y2="42.0436" width="0.254" layer="1"/>
 <wire x1="25.0124" y1="42.0436" x2="25.4" y2="41.656" width="0.254" layer="1"/>
 <via x="25.4" y="41.656" extent="1-16" drill="0.3302"/>
 <wire x1="25.4" y1="41.656" x2="23.622" y2="43.434" width="0.254" layer="16"/>
-<wire x1="23.622" y1="43.434" x2="15.748" y2="43.434" width="0.254" layer="16"/>
-<wire x1="6.858" y1="43.434" x2="6.83" y2="43.5" width="0" layer="19" extent="16-16"/>
+<wire x1="6.83" y1="43.434" x2="6.83" y2="43.5" width="0.254" layer="16"/>
 </signal>
 <signal name="NRF-IRQ">
